File: Kicad_Project/Encoder Breakout board/Encoder Breakout board.kicad_sch (KiCad schematic)
At the start: 0 parts

Commit message: Lab 2 start
Parts:
- added J1: S9B-ZR-3.4LFSN, JST_Connector:CONN9_S9B-ZR_JST, symbol JST_Connector:S9B-ZR-3.4LFSN
- added SW1: 2925, 5925_rotary:2925_ADA, symbol SP8T Rotary Switch:2925
Connections:
- new net: J1.9, SW1.1
- new net: J1.8, SW1.2
- new net: J1.7, SW1.3
- new net: J1.6, SW1.4
- new net: J1.5, SW1.5
- new net: J1.4, SW1.6
- new net: J1.3, SW1.7
- new net: J1.2, SW1.8
- new net: J1.1, SW1.A
