File: Kicad_Project/Encoder Breakout board/Encoder Breakout board.kicad_pcb (KiCad board)
At the start: 2 copper layers, 2 parts, among them J1 S9B-ZR-3.4LFSN, SW1 2925

Commit message: PCB
Some how I havent pushed this yet
Other:
- board outline added: 24.4 x 31.8 mm
Changed lines of the file:
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@@
 	)
 	(setup
+		(stackup
+			(layer "F.SilkS"
+				(type "Top Silk Screen")
+			)
+			(layer "F.Paste"
+				(type "Top Solder Paste")
+			)
+			(layer "F.Mask"
+				(type "Top Solder Mask")
+				(thickness 0.01)
+			)
+			(layer "F.Cu"
+				(type "copper")
+				(thickness 0.035)
+			)
+			(layer "dielectric 1"
+				(type "core")
+				(thickness 1.51)
+				(material "FR4")
+				(epsilon_r 4.5)
+				(loss_tangent 0.02)
+			)
+			(layer "B.Cu"
+				(type "copper")
+				(thickness 0.035)
+			)
+			(layer "B.Mask"
+				(type "Bottom Solder Mask")
+				(thickness 0.01)
+			)
+			(layer "B.Paste"
+				(type "Bottom Solder Paste")
+			)
+			(layer "B.SilkS"
+				(type "Bottom Silk Screen")
+			)
+			(copper_finish "None")
+			(dielectric_constraints no)
+		)
 		(pad_to_mask_clearance 0)
 		(allow_soldermask_bridges_in_footprints no)
@@
 			(outputformat 1)
 			(mirror no)
-			(drillshape 1)
+			(drillshape 0)
 			(scaleselection 1)
-			(outputdirectory "")
+			(outputdirectory "./")
 		)
 	)
@@
 		(tags "S9B-ZR-3.4LFSN ")
 		(property "Reference" "J1"
-			(at 6.000001 0 180)
+			(at 6 2 180)
 			(unlocked yes)
 			(layer "F.SilkS")
@@
 		(pad "1" thru_hole circle
 			(at 0 0 180)
-			(size 1.2192 1.2192)
-			(drill 0.7112)
+			(size 1.2 1.2)
+			(drill 0.7)
 			(layers "*.Cu" "*.Mask")
 			(remove_unused_layers no)
@@
 		(pad "2" thru_hole circle
 			(at 1.5 0 180)
-			(size 1.2192 1.2192)
-			(drill 0.7112)
+			(size 1.2 1.2)
+			(drill 0.7)
 			(layers "*.Cu" "*.Mask")
 			(remove_unused_layers no)
@@
 		(pad "3" thru_hole circle
 			(at 3.000002 0 180)
-			(size 1.2192 1.2192)
-			(drill 0.7112)
+			(size 1.2 1.2)
+			(drill 0.7)
 			(layers "*.Cu" "*.Mask")
 			(remove_unused_layers no)
@@
 		(pad "4" thru_hole circle
 			(at 4.500001 0 180)
-			(size 1.2192 1.2192)
-			(drill 0.7112)
+			(size 1.2 1.2)
+			(drill 0.7)
 			(layers "*.Cu" "*.Mask")
 			(remove_unused_layers no)
@@
 		(pad "5" thru_hole circle
 			(at 6.000001 0 180)
-			(size 1.2192 1.2192)
-			(drill 0.7112)
+			(size 1.2 1.2)
+			(drill 0.7)
 			(layers "*.Cu" "*.Mask")
 			(remove_unused_layers no)
@@
 		(pad "6" thru_hole circle
 			(at 7.5 0 180)
-			(size 1.2192 1.2192)
-			(drill 0.7112)
+			(size 1.2 1.2)
+			(drill 0.7)
 			(layers "*.Cu" "*.Mask")
 			(remove_unused_layers no)
@@
 		(pad "7" thru_hole circle
 			(at 9 0 180)
-			(size 1.2192 1.2192)
-			(drill 0.7112)
+			(size 1.2 1.2)
+			(drill 0.7)
 			(layers "*.Cu" "*.Mask")
 			(remove_unused_layers no)
@@
 		(pad "8" thru_hole circle
 			(at 10.500002 0 180)
-			(size 1.2192 1.2192)
-			(drill 0.7112)
+			(size 1.2 1.2)
+			(drill 0.7)
 			(layers "*.Cu" "*.Mask")
 			(remove_unused_layers no)
@@
 		(pad "9" thru_hole circle
 			(at 12.000002 0 180)
-			(size 1.2192 1.2192)
-			(drill 0.7112)
+			(size 1.2 1.2)
+			(drill 0.7)
 			(layers "*.Cu" "*.Mask")
 			(remove_unused_layers no)
@@
 		(embedded_fonts no)
 	)
+	(gr_line
+		(start 135.509 63.5)
+		(end 117.475 63.5)
+		(stroke
+			(width 0.05)
+			(type default)
+		)
+		(layer "Edge.Cuts")
+	)
+	(gr_arc
+		(start 138.684 60.325)
+		(mid 137.754064 62.570064)
+		(end 135.509 63.5)
+		(stroke
+			(width 0.05)
+			(type default)
+		)
+		(layer "Edge.Cuts")
+	)
+	(gr_arc
+		(start 135.509 31.75)
+		(mid 137.754064 32.679936)
+		(end 138.684 34.925)
+		(stroke
+			(width 0.05)
+			(type default)
+		)
+		(layer "Edge.Cuts")
+	)
+	(gr_line
+		(start 117.475 31.75)
+		(end 135.509 31.75)
+		(stroke
+			(width 0.05)
+			(type default)
+		)
+		(layer "Edge.Cuts")
+	)
+	(gr_line
+		(start 114.3 60.325)
+		(end 114.3 34.925)
+		(stroke
+			(width 0.05)
+			(type default)
+		)
+		(layer "Edge.Cuts")
+	)
+	(gr_line
+		(start 138.684 34.925)
+		(end 138.684 60.325)
+		(stroke
+			(width 0.05)
+			(type default)
+		)
+		(layer "Edge.Cuts")
+	)
+	(gr_arc
+		(start 114.3 34.925)
+		(mid 115.229936 32.679936)
+		(end 117.475 31.75)
+		(stroke
+			(width 0.05)
+			(type default)
+		)
+		(layer "Edge.Cuts")
+	)
+	(gr_arc
+		(start 117.475 63.5)
+		(mid 115.229936 62.570064)
+		(end 114.3 60.325)
+		(stroke
+			(width 0.05)
+			(type default)
+		)
+		(layer "Edge.Cuts")
+	)
 	(segment
